Commit message: www1

File: install/antbot_description/share/antbot_description/urdf/antbot.urdf.xacro (robot description, xacro)
@@ -1,4 +1,6 @@
 <?xml version="1.0"?>
 <robot xmlns:xacro="http://ros.org/wiki/xacro" name="antbot">
+  <!-- ===== Include: Lidar macro ===== -->
+  <xacro:include filename="$(find antbot_description)/urdf/sensors/antbot_lidar.xacro"/>
   <!-- ===== Params ===== -->
   <!-- ยกฐานจากพื้นเพิ่ม เพื่อลดการลากพื้น -->
@@ -265,25 +267,18 @@
     <origin xyz="0 0 0.12"/>
   </joint>
-  <link name="lidar_link">
-    <visual>
-      <origin xyz="0 0 0.02"/>
-      <geometry>
-        <mesh filename="${mesh_path}/lidar.stl"/>
-      </geometry>
-      <material name="red">
-        <color rgba="0.9 0.1 0.1 1"/>
-      </material>
-    </visual>
-    <inertial>
-      <mass value="${lidar_mass}"/>
-      <origin xyz="0 0 0"/>
-      <inertia ixx="0.0001" ixy="0" ixz="0" iyy="0.0001" iyz="0" izz="0.0001"/>
-    </inertial>
-  </link>
-  <joint name="lidar_joint" type="fixed">
-    <parent link="pillar_link"/>
-    <child  link="lidar_link"/>
-    <origin xyz="0 0 0.1"/>
-  </joint>
+  <!-- ===== LIDAR (แทนที่บล็อก mesh เดิมด้วย macro ที่มี sensor) ===== -->
+  <xacro:antbot_lidar
+      parent="pillar_link"
+      z="0.10"
+      topic="/scan"
+      frame_id="lidar_link"
+      update_rate="10"
+      samples="360"
+      resolution="1"
+      min_angle="-3.14159"
+      max_angle="3.14159"
+      range_min="0.2"
+      range_max="12.0"
+      noise_stddev="0.01"/>
   <link name="omron_link">
     <visual>

Commit message: first commit

File: install/antbot_description/share/antbot_description/urdf/antbot.urdf.xacro (robot description, xacro)
@@ -1,19 +1,22 @@
 <?xml version="1.0"?>
 <robot xmlns:xacro="http://ros.org/wiki/xacro" name="antbot">
-  <!-- ===== Include: Lidar macro ===== -->
+  <!-- Includes -->
+   <!-- รวมมาโคร LiDAR -->
   <xacro:include filename="$(find antbot_description)/urdf/sensors/antbot_lidar.xacro"/>
+  <!-- รวมมาโคร IMU -->
+  <xacro:include filename="$(find antbot_description)/urdf/sensors/antbot_imu.xacro"/>
+   <!-- ✅ รวมมาโคร Ultrasonic -->
+  <xacro:include filename="$(find antbot_description)/urdf/sensors/antbot_ultrasonic.xacro"/>
   <!-- ===== Params ===== -->
-  <!-- ยกฐานจากพื้นเพิ่ม เพื่อลดการลากพื้น -->
-  <xacro:property name="base_clearance" value="0.03"/>  <!-- ~3 ซม. -->
+  <xacro:arg name="ctrl_yaml" default=""/>
+  <xacro:property name="base_clearance" value="0.03"/>
   <xacro:property name="mesh_path"    value="package://antbot_description/meshes"/>
-  <xacro:property name="wheel_radius" value="0.08"/>   <!-- 8 cm -->
-  <xacro:property name="wheel_width"  value="0.06"/>   <!-- 6 cm -->
-  <!-- ขนาดกล่องแทนฐาน -->
+  <xacro:property name="wheel_radius" value="0.08"/>
+  <xacro:property name="wheel_width"  value="0.06"/>
   <xacro:property name="base_size_x" value="0.55"/>
   <xacro:property name="base_size_y" value="0.42"/>
   <xacro:property name="base_size_z" value="0.10"/>
-  <!-- มวลสมเหตุสมผล -->
-  <xacro:property name="base_mass"   value="5.0"/>   <!-- ~12 kg -->
-  <xacro:property name="wheel_mass"  value="1.00"/>  <!-- ~1 kg/ล้อ -->
+  <xacro:property name="base_mass"   value="5.0"/>
+  <xacro:property name="wheel_mass"  value="1.0"/>
   <xacro:property name="frame_mass"  value="0.10"/>
   <xacro:property name="pillar_mass" value="0.20"/>
@@ -21,6 +24,9 @@
   <xacro:property name="omron_mass"  value="0.10"/>
   <xacro:property name="steer_mass"  value="0.05"/>
-  <!-- ===== Macros: inertia ให้ถูกฟิสิกส์ ===== -->
-  <!-- กล่อง: ขยับจุดมวลให้ตรงกับ collision -->
+  <!-- จุดติดตั้งหัว LiDAR -->
+  <xacro:property name="lidar_x" value="-0.013"/>
+  <xacro:property name="lidar_y" value="0.063"/>
+  <xacro:property name="lidar_z" value="0.613"/>
+  <!-- ===== inertia helpers ===== -->
   <xacro:macro name="inertial_box" params="mass x y z ox oy oz">
     <inertial>
@@ -33,10 +39,8 @@
     </inertial>
   </xacro:macro>
-  <!-- ทรงกระบอกแกน X (ล้อหมุนรอบแกน X) -->
   <xacro:macro name="inertial_cyl_x" params="mass r l">
     <inertial>
       <mass value="${mass}"/>
       <origin xyz="0 0 0"/>
-      <!-- Ixx = 1/2 m r^2 ; Iyy=Izz = 1/12 m(3r^2 + l^2) -->
       <inertia
         ixx="${0.5*mass*r*r}" ixy="0" ixz="0"
@@ -48,67 +52,37 @@
   <link name="base_link">
     <visual>
-      <origin xyz="0 0 0" rpy="0 0 0"/>
-      <geometry>
-        <mesh filename="${mesh_path}/antbot_base.stl"/>
-      </geometry>
-      <material name="gray">
-        <color rgba="0.6 0.6 0.6 1"/>
-      </material>
-    </visual>
-    <!-- collision เป็นกล่อง และยกขึ้นครึ่งความหนา + ระยะเผื่อ -->
+      <origin xyz="0 0 0" rpy="0 0 1.57079632679"/>
+      <geometry><mesh filename="${mesh_path}/antbot_base.stl"/></geometry>
+      <material name="gray"><color rgba="0.6 0.6 0.6 1"/></material>
+    </visual>
     <collision name="base_link_collision">
       <origin xyz="0 0 ${base_size_z/2.0 + base_clearance}" rpy="0 0 0"/>
-      <geometry>
-        <box size="${base_size_x} ${base_size_y} ${base_size_z}"/>
-      </geometry>
-      <!-- ลด friction ของฐานเพื่อลดแรงต้านเมื่อเผลอแตะพื้น -->
-      <surface>
-        <friction>
-          <ode>
-            <mu>0.3</mu>
-            <mu2>0.3</mu2>
-          </ode>
-        </friction>
-      </surface>
-    </collision>
-    <!-- inertial ตรงกับ collision -->
-    <xacro:inertial_box
-      mass="${base_mass}"
-      x="${base_size_x}"
-      y="${base_size_y}"
-      z="${base_size_z}"
+      <geometry><box size="${base_size_x} ${base_size_y} ${base_size_z}"/></geometry>
+      <surface><friction><ode><mu>0.3</mu><mu2>0.3</mu2></ode></friction></surface>
+    </collision>
+    <xacro:inertial_box mass="${base_mass}"
+      x="${base_size_x}" y="${base_size_y}" z="${base_size_z}"
       ox="0" oy="0" oz="${base_size_z/2.0 + base_clearance}"/>
   </link>
-  <!-- ===== Rear Left Wheel ===== -->
+  <!-- ===== ติดตั้ง IMU ให้ลอยเหนือฐานเล็กน้อย ===== -->
+  <xacro:antbot_imu
+    parent="base_link"
+    frame_id="imu_link"
+    xyz_offset="0 0 0.959"
+    rpy_offset="0 0 0"
+    update_rate="100.0"/>
+  <!-- ===== Wheels ===== -->
   <link name="wheel_rear_left_link">
     <visual>
       <origin xyz="0 0 0"/>
-      <geometry>
-        <mesh filename="${mesh_path}/wheel_rear_centered_clean.stl"/>
-      </geometry>
-      <material name="black">
-        <color rgba="0.1 0.1 0.1 1"/>
-      </material>
-    </visual>
-    <!-- cylinder แกน X -->
+      <geometry><mesh filename="${mesh_path}/wheel_rear_centered_clean.stl"/></geometry>
+      <material name="black"><color rgba="0.1 0.1 0.1 1"/></material>
+    </visual>
     <collision name="wheel_rear_left_link_collision">
       <origin xyz="0 0 0" rpy="0 1.57079632679 0"/>
-      <geometry>
-        <cylinder radius="${wheel_radius}" length="${wheel_width}"/>
-      </geometry>
+      <geometry><cylinder radius="${wheel_radius}" length="${wheel_width}"/></geometry>
       <surface>
-        <friction>
-          <ode>
-            <mu>1.8</mu>
-            <mu2>1.8</mu2>
-          </ode>
-        </friction>
-        <!-- contact แข็งขึ้น ลดอาการเด้ง/ลื่น -->
-        <contact>
-          <ode>
-            <kp>1e7</kp>
-            <kd>1e5</kd>
-          </ode>
-        </contact>
+        <friction><ode><mu>1.8</mu><mu2>1.8</mu2></ode></friction>
+        <contact><ode><kp>1e7</kp><kd>1e5</kd></ode></contact>
       </surface>
     </collision>
@@ -116,42 +90,21 @@
   </link>
   <joint name="wheel_rear_left_joint" type="continuous">
-    <parent link="base_link"/>
-    <child  link="wheel_rear_left_link"/>
-    <origin xyz="0.285 0.5 ${wheel_radius}" rpy="0 0 0"/>
-    <axis xyz="1 0 0"/>
-    <!-- ลดแดมป์ให้ล้อขึ้นรอบไว -->
-    <dynamics damping="0.001" friction="0.0"/>
-    <!-- เพิ่มเพดานแรง/ความเร็ว -->
+    <parent link="base_link"/><child link="wheel_rear_left_link"/>
+    <origin xyz="-0.497 0.28 ${wheel_radius}" rpy="0 0 1.57079632679"/>
+    <axis xyz="1 0 0"/><dynamics damping="0.001" friction="0.0"/>
     <limit effort="80.0" velocity="120.0"/>
   </joint>
-  <!-- ===== Rear Right Wheel ===== -->
   <link name="wheel_rear_right_link">
     <visual>
       <origin xyz="0 0 0"/>
-      <geometry>
-        <mesh filename="${mesh_path}/wheel_rear_centered_clean.stl"/>
-      </geometry>
-      <material name="black">
-        <color rgba="0.1 0.1 0.1 1"/>
-      </material>
+      <geometry><mesh filename="${mesh_path}/wheel_rear_centered_clean.stl"/></geometry>
+      <material name="black"><color rgba="0.1 0.1 0.1 1"/></material>
     </visual>
     <collision name="wheel_rear_right_link_collision">
       <origin xyz="0 0 0" rpy="0 1.57079632679 0"/>
-      <geometry>
-        <cylinder radius="${wheel_radius}" length="${wheel_width}"/>
-      </geometry>
+      <geometry><cylinder radius="${wheel_radius}" length="${wheel_width}"/></geometry>
       <surface>
-        <friction>
-          <ode>
-            <mu>1.8</mu>
-            <mu2>1.8</mu2>
-          </ode>
-        </friction>
-        <contact>
-          <ode>
-            <kp>1e7</kp>
-            <kd>1e5</kd>
-          </ode>
-        </contact>
+        <friction><ode><mu>1.8</mu><mu2>1.8</mu2></ode></friction>
+        <contact><ode><kp>1e7</kp><kd>1e5</kd></ode></contact>
       </surface>
     </collision>
@@ -159,57 +112,35 @@
   </link>
   <joint name="wheel_rear_right_joint" type="continuous">
-    <parent link="base_link"/>
-    <child  link="wheel_rear_right_link"/>
-    <origin xyz="-0.245 0.5 ${wheel_radius}" rpy="0 0 0"/>
-    <axis xyz="1 0 0"/>
-    <dynamics damping="0.001" friction="0.0"/>
+    <parent link="base_link"/><child link="wheel_rear_right_link"/>
+    <origin xyz="-0.50 -0.23 ${wheel_radius}" rpy="0 0 1.57079632679"/>
+    <axis xyz="1 0 0"/><dynamics damping="0.001" friction="0.0"/>
     <limit effort="80.0" velocity="120.0"/>
   </joint>
-  <!-- ===== Steering ===== -->
+  <!-- ===== Steering + front wheel ===== -->
   <link name="steering_link">
     <inertial>
-      <mass value="${steer_mass}"/>
-      <origin xyz="0 0 0"/>
+      <mass value="${steer_mass}"/><origin xyz="0 0 0"/>
       <inertia ixx="0.0001" ixy="0" ixz="0" iyy="0.0001" iyz="0" izz="0.0001"/>
     </inertial>
   </link>
   <joint name="steering_joint" type="revolute">
-    <parent link="base_link"/>
-    <child  link="steering_link"/>
-    <origin xyz="0.07 -0.04 ${wheel_radius}" rpy="0 0 0"/>
+    <parent link="base_link"/><child link="steering_link"/>
+    <origin xyz="0.035 0.11 ${wheel_radius}" rpy="0 0 1.57079632679"/>
     <axis xyz="0 0 1"/>
-    <!-- ลดแดมป์เพื่อให้เลี้ยวตอบสนองไวขึ้น -->
-    <dynamics damping="0.05" friction="0.0"/>
-    <limit effort="12.0" velocity="12.0" lower="-0.6" upper="0.6"/>
-  </joint>
-  <!-- ===== Front Wheel ===== -->
+    <dynamics damping="2.0" friction="0.0"/>
+    <limit effort="8.0" velocity="1.8" lower="-0.62" upper="0.62"/>
+  </joint>
   <link name="wheel_front_link">
     <visual>
       <origin xyz="0 0 0"/>
-      <geometry>
-        <mesh filename="${mesh_path}/wheel_front_centered.stl"/>
-      </geometry>
-      <material name="black">
-        <color rgba="0.1 0.1 0.1 1"/>
-      </material>
+      <geometry><mesh filename="${mesh_path}/wheel_front_centered.stl"/></geometry>
+      <material name="black"><color rgba="0.1 0.1 0.1 1"/></material>
     </visual>
     <collision name="wheel_front_link_collision">
       <origin xyz="0 0 0" rpy="0 1.57079632679 0"/>
-      <geometry>
-        <cylinder radius="${wheel_radius}" length="${wheel_width}"/>
-      </geometry>
+      <geometry><cylinder radius="${wheel_radius}" length="${wheel_width}"/></geometry>
       <surface>
-        <friction>
-          <ode>
-            <mu>1.8</mu>
-            <mu2>1.8</mu2>
-          </ode>
-        </friction>
-        <contact>
-          <ode>
-            <kp>1e7</kp>
-            <kd>1e5</kd>
-          </ode>
-        </contact>
+        <friction><ode><mu>1.8</mu><mu2>1.8</mu2></ode></friction>
+        <contact><ode><kp>1e7</kp><kd>1e5</kd></ode></contact>
       </surface>
     </collision>
@@ -217,88 +148,112 @@
   </link>
   <joint name="front_wheel_joint" type="continuous">
-    <parent link="steering_link"/>
-    <child  link="wheel_front_link"/>
+    <parent link="steering_link"/><child link="wheel_front_link"/>
     <origin xyz="-0.051 0.005 0" rpy="0 0 0"/>
-    <axis xyz="1 0 0"/>
-    <dynamics damping="0.001" friction="0.0"/>
+    <axis xyz="1 0 0"/><dynamics damping="0.001" friction="0.0"/>
     <limit effort="80.0" velocity="120.0"/>
   </joint>
-  <!-- ===== Decorative / extra links ===== -->
+  <!-- ===== Extra visuals ===== -->
   <link name="wheel_front_frame_link">
     <visual>
       <origin xyz="0 -0.13 -0.05"/>
-      <geometry>
-        <mesh filename="${mesh_path}/wheel_front_frame.stl"/>
-      </geometry>
-      <material name="gray">
-        <color rgba="0.5 0.5 0.5 1"/>
-      </material>
-    </visual>
-    <inertial>
-      <mass value="${frame_mass}"/>
-      <origin xyz="0 0 0"/>
+      <geometry><mesh filename="${mesh_path}/wheel_front_frame.stl"/></geometry>
+      <material name="gray"><color rgba="0.5 0.5 0.5 1"/></material>
+    </visual>
+    <inertial>
+      <mass value="${frame_mass}"/><origin xyz="0 0 0"/>
       <inertia ixx="0.0001" ixy="0" ixz="0" iyy="0.0001" iyz="0" izz="0.0001"/>
     </inertial>
   </link>
   <joint name="wheel_front_frame_joint" type="fixed">
-    <parent link="steering_link"/>
-    <child  link="wheel_front_frame_link"/>
+    <parent link="steering_link"/><child link="wheel_front_frame_link"/>
     <origin xyz="-0.12 0.175 -0.0258"/>
   </joint>
+  <!-- ===== Pillar ===== -->
   <link name="pillar_link">
     <visual>
-      <origin xyz="0 0 0.12"/>
-      <geometry>
-        <mesh filename="${mesh_path}/pillar.stl"/>
-      </geometry>
-      <material name="gray">
-        <color rgba="0.6 0.6 0.6 1"/>
-      </material>
-    </visual>
-    <inertial>
-      <mass value="${pillar_mass}"/>
-      <origin xyz="0 0 0"/>
+      <origin xyz="0 0 0"/>
+      <geometry><mesh filename="${mesh_path}/pillar_centered_origin.stl"/></geometry>
+      <material name="gray"><color rgba="0.6 0.6 0.6 1"/></material>
+    </visual>
+    <inertial>
+      <mass value="${pillar_mass}"/><origin xyz="0 0 0"/>
       <inertia ixx="0.0002" ixy="0" ixz="0" iyy="0.0002" iyz="0" izz="0.0002"/>
     </inertial>
   </link>
   <joint name="pillar_joint" type="fixed">
-    <parent link="base_link"/>
-    <child  link="pillar_link"/>
-    <origin xyz="0 0 0.12"/>
-  </joint>
-  <!-- ===== LIDAR (แทนที่บล็อก mesh เดิมด้วย macro ที่มี sensor) ===== -->
-  <xacro:antbot_lidar
-      parent="pillar_link"
-      z="0.10"
-      topic="/scan"
-      frame_id="lidar_link"
-      update_rate="10"
-      samples="360"
-      resolution="1"
-      min_angle="-3.14159"
-      max_angle="3.14159"
-      range_min="0.2"
-      range_max="12.0"
-      noise_stddev="0.01"/>
+    <parent link="base_link"/><child link="pillar_link"/>
+    <origin xyz="-0.4936 0.025 1.1917" rpy="0 0 1.57079632679"/>
+  </joint>
+  <!-- ===== LiDAR head ===== -->
+  <link name="lidar_link">
+    <visual>
+      <origin xyz="0 0 0.02"/>
+      <geometry><mesh filename="${mesh_path}/lidar_centered_origin.stl"/></geometry>
+      <material name="red"><color rgba="0.9 0.1 0.1 1"/></material>
+    </visual>
+    <inertial>
+      <mass value="${lidar_mass}"/>
+      <origin xyz="0 0 0"/>
+      <inertia ixx="0.0001" ixy="0" ixz="0" iyy="0.0001" iyz="0" izz="0.0001"/>
+    </inertial>
+  </link>
+  <joint name="lidar_joint" type="fixed">
+    <parent link="pillar_link"/><child link="lidar_link"/>
+    <origin xyz="${lidar_x} ${lidar_y} ${lidar_z}" rpy="0 0 0"/>
+  </joint>
+  <!-- กรอบเซนเซอร์ LiDAR -->
+  <link name="lidar_sensor_link"/>
+  <joint name="lidar_sensor_joint" type="fixed">
+    <parent link="lidar_link"/>
+    <child  link="lidar_sensor_link"/>
+    <origin xyz="0 0 0" rpy="0 0 0"/>
+  </joint>
+  <!-- ผูกปลั๊กอิน LiDAR -->
+  <xacro:antbot_lidar_attach
+    link="lidar_sensor_link"
+    topic="/scan"
+    frame_id="lidar_sensor_link"
+    update_rate="15"
+    visualize="true"
+    samples="720"
+    resolution="1"
+    min_angle="-3.14159"
+    max_angle="3.14159"
+    vertical_samples="1"
+    vertical_resolution="1"
+    vertical_min_angle="0"
+    vertical_max_angle="0"
+    range_min="0.15"
+    range_max="8.0"
+    noise_stddev="0.003"/>
+  <!-- ===== Ultrasonic (หน้ากลาง) ===== -->
+  <xacro:antbot_ultrasonic
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